File: PCB_Init/PCB_Init.sch (KiCad schematic (older format))
At the start: 33 parts

Commit message: Added KiCAD file with AtMega2560 details and pulse oxi 2
Parts:
- removed J?: Conn_01x07, symbol Connector_Generic:Conn_01x07
- removed U?: AMS1117CD-1.8, Package_TO_SOT_SMD:TO-252-3_TabPin2, symbol Regulator_Linear:AMS1117CD-1.8
Changed lines of the file:
@@
 $EndComp
 $Comp
-L power:GND #PWR?
+L power:GND #PWR0101
 U 1 1 6070FA31
 P 2600 1700
-F 0 "#PWR?" H 2600 1450 50  0001 C CNN
+F 0 "#PWR0101" H 2600 1450 50  0001 C CNN
 F 1 "GND" H 2605 1527 50  0000 C CNN
 F 2 "" H 2600 1700 50  0001 C CNN
@@
 $EndComp
 $Comp
-L power:GND #PWR?
+L power:GND #PWR0102
 U 1 1 60710E78
 P 3200 1700
-F 0 "#PWR?" H 3200 1450 50  0001 C CNN
+F 0 "#PWR0102" H 3200 1450 50  0001 C CNN
 F 1 "GND" H 3205 1527 50  0000 C CNN
 F 2 "" H 3200 1700 50  0001 C CNN
@@
 $EndComp
 $Comp
-L power:GND #PWR?
+L power:GND #PWR0103
 U 1 1 607118F1
 P 1500 1700
-F 0 "#PWR?" H 1500 1450 50  0001 C CNN
+F 0 "#PWR0103" H 1500 1450 50  0001 C CNN
 F 1 "GND" H 1505 1527 50  0000 C CNN
 F 2 "" H 1500 1700 50  0001 C CNN
@@
 $EndComp
 $Comp
-L power:GND #PWR?
+L power:GND #PWR0104
 U 1 1 6072386B
 P 9200 4800
-F 0 "#PWR?" H 9200 4550 50  0001 C CNN
+F 0 "#PWR0104" H 9200 4550 50  0001 C CNN
 F 1 "GND" V 9205 4672 50  0000 R CNN
 F 2 "" H 9200 4800 50  0001 C CNN
@@
 $EndComp
 $Comp
-L power:+12V #PWR?
+L power:+12V #PWR0105
 U 1 1 6073258E
 P 1500 750
-F 0 "#PWR?" H 1500 600 50  0001 C CNN
+F 0 "#PWR0105" H 1500 600 50  0001 C CNN
 F 1 "+12V" H 1515 923 50  0000 C CNN
 F 2 "" H 1500 750 50  0001 C CNN
@@
 $EndComp
 $Comp
-L power:+12V #PWR?
+L power:+12V #PWR0106
 U 1 1 607334A8
 P 2600 750
-F 0 "#PWR?" H 2600 600 50  0001 C CNN
+F 0 "#PWR0106" H 2600 600 50  0001 C CNN
 F 1 "+12V" H 2615 923 50  0000 C CNN
 F 2 "" H 2600 750 50  0001 C CNN
@@
 $EndComp
 $Comp
-L power:+5V #PWR?
+L power:+5V #PWR0107
 U 1 1 60734807
 P 3200 750
-F 0 "#PWR?" H 3200 600 50  0001 C CNN
+F 0 "#PWR0107" H 3200 600 50  0001 C CNN
 F 1 "+5V" H 3215 923 50  0000 C CNN
 F 2 "" H 3200 750 50  0001 C CNN
@@
 $EndComp
 $Comp
-L power:GND #PWR?
+L power:GND #PWR0108
 U 1 1 60734FB9
 P 2900 1700
-F 0 "#PWR?" H 2900 1450 50  0001 C CNN
+F 0 "#PWR0108" H 2900 1450 50  0001 C CNN
 F 1 "GND" H 2905 1527 50  0000 C CNN
 F 2 "" H 2900 1700 50  0001 C CNN
@@
 	9600 4800 9500 4800
 $Comp
-L power:GND #PWR?
+L power:GND #PWR0109
 U 1 1 607245A0
 P 9600 4200
-F 0 "#PWR?" H 9600 3950 50  0001 C CNN
+F 0 "#PWR0109" H 9600 3950 50  0001 C CNN
 F 1 "GND" H 9605 4027 50  0000 C CNN
 F 2 "" H 9600 4200 50  0001 C CNN
@@
 $EndComp
 $Comp
-L power:GND #PWR?
+L power:GND #PWR0110
 U 1 1 6071D006
 P 9750 2700
-F 0 "#PWR?" H 9750 2450 50  0001 C CNN
+F 0 "#PWR0110" H 9750 2450 50  0001 C CNN
 F 1 "GND" V 9755 2572 50  0000 R CNN
 F 2 "" H 9750 2700 50  0001 C CNN
@@
 $EndComp
 $Comp
-L power:GND #PWR?
+L power:GND #PWR0111
 U 1 1 60712D07
 P 3300 5550
-F 0 "#PWR?" H 3300 5300 50  0001 C CNN
+F 0 "#PWR0111" H 3300 5300 50  0001 C CNN
 F 1 "GND" H 3305 5377 50  0000 C CNN
 F 2 "" H 3300 5550 50  0001 C CNN
@@
 $EndComp
 $Comp
-L power:GND #PWR?
+L power:GND #PWR0112
 U 1 1 60713D28
 P 2500 5550
-F 0 "#PWR?" H 2500 5300 50  0001 C CNN
+F 0 "#PWR0112" H 2500 5300 50  0001 C CNN
 F 1 "GND" H 2505 5377 50  0000 C CNN
 F 2 "" H 2500 5550 50  0001 C CNN
@@
 $EndComp
 $Comp
-L power:GND #PWR?
+L power:GND #PWR0113
 U 1 1 607146B8
 P 1850 5550
-F 0 "#PWR?" H 1850 5300 50  0001 C CNN
+F 0 "#PWR0113" H 1850 5300 50  0001 C CNN
 F 1 "GND" H 1855 5377 50  0000 C CNN
 F 2 "" H 1850 5550 50  0001 C CNN
@@
 $EndComp
 $Comp
-L power:GND #PWR?
+L power:GND #PWR0114
 U 1 1 60714FCA
 P 1150 5550
-F 0 "#PWR?" H 1150 5300 50  0001 C CNN
+F 0 "#PWR0114" H 1150 5300 50  0001 C CNN
 F 1 "GND" H 1155 5377 50  0000 C CNN
 F 2 "" H 1150 5550 50  0001 C CNN
@@
 $EndComp
 $Comp
-L power:GND #PWR?
+L power:GND #PWR0115
 U 1 1 607251CA
 P 850 5400
-F 0 "#PWR?" H 850 5150 50  0001 C CNN
+F 0 "#PWR0115" H 850 5150 50  0001 C CNN
 F 1 "GND" H 855 5227 50  0000 C CNN
 F 2 "" H 850 5400 50  0001 C CNN
@@
 $EndComp
 $Comp
-L power:GND #PWR?
+L power:GND #PWR0116
 U 1 1 60725EBC
 P 1550 5400
-F 0 "#PWR?" H 1550 5150 50  0001 C CNN
+F 0 "#PWR0116" H 1550 5150 50  0001 C CNN
 F 1 "GND" H 1555 5227 50  0000 C CNN
 F 2 "" H 1550 5400 50  0001 C CNN
@@
 $EndComp
 $Comp
-L power:GND #PWR?
+L power:GND #PWR0117
 U 1 1 60726AEB
 P 2200 5400
-F 0 "#PWR?" H 2200 5150 50  0001 C CNN
+F 0 "#PWR0117" H 2200 5150 50  0001 C CNN
 F 1 "GND" H 2205 5227 50  0000 C CNN
 F 2 "" H 2200 5400 50  0001 C CNN
@@
 $EndComp
 $Comp
-L power:GND #PWR?
+L power:GND #PWR0118
 U 1 1 60727ED0
 P 3000 5400
-F 0 "#PWR?" H 3000 5150 50  0001 C CNN
+F 0 "#PWR0118" H 3000 5150 50  0001 C CNN
 F 1 "GND" H 3005 5227 50  0000 C CNN
 F 2 "" H 3000 5400 50  0001 C CNN
@@
 	850  5100 850  4900
 $Comp
-L power:+5V #PWR?
+L power:+5V #PWR0119
 U 1 1 606C4D8A
 P 4100 5500
-F 0 "#PWR?" H 4100 5350 50  0001 C CNN
+F 0 "#PWR0119" H 4100 5350 50  0001 C CNN
 F 1 "+5V" H 4115 5673 50  0000 C CNN
 F 2 "" H 4100 5500 50  0001 C CNN
@@
 $EndComp
 $Comp
-L power:+5V #PWR?
+L power:+5V #PWR0120
 U 1 1 606C81FB
 P 4700 5500
-F 0 "#PWR?" H 4700 5350 50  0001 C CNN
+F 0 "#PWR0120" H 4700 5350 50  0001 C CNN
 F 1 "+5V" H 4715 5673 50  0000 C CNN
 F 2 "" H 4700 5500 50  0001 C CNN
@@
 $EndComp
 $Comp
-L power:+5V #PWR?
+L power:+5V #PWR0121
 U 1 1 606C8AFD
 P 5400 5500
-F 0 "#PWR?" H 5400 5350 50  0001 C CNN
+F 0 "#PWR0121" H 5400 5350 50  0001 C CNN
 F 1 "+5V" H 5415 5673 50  0000 C CNN
 F 2 "" H 5400 5500 50  0001 C CNN
@@
 $EndComp
 $Comp
-L power:+5V #PWR?
+L power:+5V #PWR0122
 U 1 1 606C9370
 P 6000 5500
-F 0 "#PWR?" H 6000 5350 50  0001 C CNN
+F 0 "#PWR0122" H 6000 5350 50  0001 C CNN
 F 1 "+5V" H 6015 5673 50  0000 C CNN
 F 2 "" H 6000 5500 50  0001 C CNN
@@
 $EndComp
 $Comp
-L power:GND #PWR?
+L power:GND #PWR0123
 U 1 1 606C9B0F
 P 3800 5500
-F 0 "#PWR?" H 3800 5250 50  0001 C CNN
+F 0 "#PWR0123" H 3800 5250 50  0001 C CNN
 F 1 "GND" H 3805 5327 50  0000 C CNN
 F 2 "" H 3800 5500 50  0001 C CNN
@@
 $EndComp
 $Comp
-L power:GND #PWR?
+L power:GND #PWR0124
 U 1 1 606CA38F
 P 4400 5500
-F 0 "#PWR?" H 4400 5250 50  0001 C CNN
+F 0 "#PWR0124" H 4400 5250 50  0001 C CNN
 F 1 "GND" H 4405 5327 50  0000 C CNN
 F 2 "" H 4400 5500 50  0001 C CNN
@@
 $EndComp
 $Comp
-L power:GND #PWR?
+L power:GND #PWR0125
 U 1 1 606CAB66
 P 5100 5500
-F 0 "#PWR?" H 5100 5250 50  0001 C CNN
+F 0 "#PWR0125" H 5100 5250 50  0001 C CNN
 F 1 "GND" H 5105 5327 50  0000 C CNN
 F 2 "" H 5100 5500 50  0001 C CNN
@@
 $EndComp
 $Comp
-L power:GND #PWR?
+L power:GND #PWR0126
 U 1 1 606CB269
 P 5700 5500
-F 0 "#PWR?" H 5700 5250 50  0001 C CNN
+F 0 "#PWR0126" H 5700 5250 50  0001 C CNN
 F 1 "GND" H 5705 5327 50  0000 C CNN
 F 2 "" H 5700 5500 50  0001 C CNN
@@
 $EndComp
 $Comp
-L power:GND #PWR?
+L power:GND #PWR0127
 U 1 1 607158CF
 P 4400 1950
-F 0 "#PWR?" H 4400 1700 50  0001 C CNN
+F 0 "#PWR0127" H 4400 1700 50  0001 C CNN
 F 1 "GND" H 4405 1777 50  0000 C CNN
 F 2 "" H 4400 1950 50  0001 C CNN
@@
 $EndComp
 $Comp
-L power:GND #PWR?
+L power:GND #PWR0128
 U 1 1 60718139
 P 5700 1550
-F 0 "#PWR?" H 5700 1300 50  0001 C CNN
+F 0 "#PWR0128" H 5700 1300 50  0001 C CNN
 F 1 "GND" H 5705 1377 50  0000 C CNN
 F 2 "" H 5700 1550 50  0001 C CNN
@@
 $EndComp
 $Comp
-L power:GND #PWR?
+L power:GND #PWR0129
 U 1 1 6071858A
 P 4100 1450
-F 0 "#PWR?" H 4100 1200 50  0001 C CNN
+F 0 "#PWR0129" H 4100 1200 50  0001 C CNN
 F 1 "GND" H 4105 1277 50  0000 C CNN
 F 2 "" H 4100 1450 50  0001 C CNN
@@
 $EndComp
 $Comp
-L power:GND #PWR?
+L power:GND #PWR0130
 U 1 1 60718DAB
 P 5200 1150
-F 0 "#PWR?" H 5200 900 50  0001 C CNN
+F 0 "#PWR0130" H 5200 900 50  0001 C CNN
 F 1 "GND" H 5205 977 50  0000 C CNN
 F 2 "" H 5200 1150 50  0001 C CNN
@@
 $EndComp
 $Comp
-L power:GND #PWR?
+L power:GND #PWR0131
 U 1 1 6071B93A
 P 8650 850
-F 0 "#PWR?" H 8650 600 50  0001 C CNN
+F 0 "#PWR0131" H 8650 600 50  0001 C CNN
 F 1 "GND" H 8655 677 50  0000 C CNN
 F 2 "" H 8650 850 50  0001 C CNN
@@
 $EndComp
 $Comp
-L power:GND #PWR?
+L power:GND #PWR0132
 U 1 1 6071C568
 P 7550 850
-F 0 "#PWR?" H 7550 600 50  0001 C CNN
+F 0 "#PWR0132" H 7550 600 50  0001 C CNN
 F 1 "GND" H 7555 677 50  0000 C CNN
 F 2 "" H 7550 850 50  0001 C CNN
@@
 Buzzer
 $Comp
-L power:+5V #PWR?
+L power:+5V #PWR0133
 U 1 1 6072270A
 P 5100 750
-F 0 "#PWR?" H 5100 600 50  0001 C CNN
+F 0 "#PWR0133" H 5100 600 50  0001 C CNN
 F 1 "+5V" H 5115 923 50  0000 C CNN
 F 2 "" H 5100 750 50  0001 C CNN
@@
 ErrorLight
 $Comp
-L power:GND #PWR?
+L power:GND #PWR0134
 U 1 1 6074FCE9
 P 1400 3250
-F 0 "#PWR?" H 1400 3000 50  0001 C CNN
+F 0 "#PWR0134" H 1400 3000 50  0001 C CNN
 F 1 "GND" V 1405 3122 50  0000 R CNN
 F 2 "" H 1400 3250 50  0001 C CNN
@@
 Driver1
 $Comp
-L Connector_Generic:Conn_01x07 J?
-U 1 1 6072124E
-P 3100 11250
-F 0 "J?" H 3018 10725 50  0000 C CNN
-F 1 "Conn_01x07" H 3018 10816 50  0000 C CNN
-F 2 "" H 3100 11250 50  0001 C CNN
-F 3 "~" H 3100 11250 50  0001 C CNN
-	1    3100 11250
-	-1   0    0    1
-$EndComp
-$Comp
-L Regulator_Linear:AMS1117CD-1.8 U?
-U 1 1 6072608A
-P 6050 10550
-F 0 "U?" H 6050 10792 50  0000 C CNN
-F 1 "AMS1117CD-1.8" H 6050 10701 50  0000 C CNN
-F 2 "Package_TO_SOT_SMD:TO-252-3_TabPin2" H 6050 10750 50  0001 C CNN
-F 3 "http://www.advanced-monolithic.com/pdf/ds1117.pdf" H 6150 10300 50  0001 C CNN
-	1    6050 10550
-	1    0    0    -1
-$EndComp
-$Comp
-L power:GND #PWR?
+L power:GND #PWR0135
 U 1 1 607413CD
 P 7900 5850
-F 0 "#PWR?" H 7900 5600 50  0001 C CNN
+F 0 "#PWR0135" H 7900 5600 50  0001 C CNN
 F 1 "GND" H 7905 5677 50  0000 C CNN
 F 2 "" H 7900 5850 50  0001 C CNN

Commit message: Plotted gerber files for initial idea
Connections:
- net SCL: now also U?.43 (PD0); no longer U?.84 (PK5)
- net SDA: now also U?.44 (PD1); no longer U?.83 (PK6)
Changed lines of the file:
@@
 Text Label 7200 5350 2    50   ~ 0
 SDA
-Text Label 4500 2450 1    50   ~ 0
-SDA
 Text Label 7200 5250 2    50   ~ 0
-SCL
-Text Label 4600 2450 1    50   ~ 0
 SCL
 $Comp
@@
 	1    0    0    -1
 $EndComp
+Text Label 4200 4050 3    50   ~ 0
+SCL
+Text Label 4100 4050 3    50   ~ 0
+SDA
 $EndSCHEMATC
