File: Work Files/PCB_Init/PCB_Init.kicad_pcb (KiCad board)
At the start: 2 copper layers, 33 parts, among them J1 Conn_01x02_Female, J2 Screw_Terminal_01x02, J3 Conn_01x02_Female, J4 Conn_01x02_Female, J5 Conn_01x02_Female, J6 Conn_01x02_Female, J7 Conn_01x02_Female, SW1 SW_Push, SW2 SW_Push, SW3 SW_Push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

Commit message: Started designing PCB2
Parts:
- J1, J3, J4, J5, J6, J7: footprint Connector_PinHeader_1.27mm:PinHeader_1x02_P1.27mm_Vertical -> Connector_PinHeader_2.54mm:PinHeader_1x02_P2.54mm_Vertical

Commit message: Started designing PCB3
Parts:
- added REF**: OSHW-Logo2_14.6x12mm_Copper, Symbol:OSHW-Logo2_14.6x12mm_Copper, F.Cu at (276.9, 158.8)
- added REF**: KiCad-Logo2_5mm_SilkScreen, Symbol:KiCad-Logo2_5mm_SilkScreen, F.Cu at (148.6, 95.2)
Other:
- board outline added: 271.8 x 161.3 mm
- board text added: "Re-Vent"

Commit message: Started designing ing PCB 4
Parts:
- removed the REF** at (148.6, 95.2)
- added REF**: KiCad-Logo2_6mm_SilkScreen, Symbol:KiCad-Logo2_6mm_SilkScreen, F.Cu at (148.6, 94.0)
- SW1, SW2, SW3, SW4: footprint Button_Switch_THT:SW_PUSH-12mm -> Button_Switch_THT:SW_CW_GPTS203211B
- moved SW4 6.84 mm to (88.9, 153.7), turned to 270 degrees
- moved SW3 6.84 mm to (67.3, 153.7), turned to 270 degrees
- moved SW2 5.68 mm to (47.0, 153.7), turned to 270 degrees
- moved SW1 5.68 mm to (26.7, 153.7), turned to 270 degrees
- moved REF** 3.59 mm to (274.3, 156.2)
- moved C3 0.36 mm to (33.0, 144.8)
- turned J1 to 180 degrees
- turned J3 to 180 degrees
- turned J4 to 180 degrees
- turned J5 to 180 degrees
Connections:
- C3 pad 1: GND -> Net-(C3-Pad1)
- C3 pad 2: Net-(C3-Pad2) -> GND
- C4 pad 1: GND -> Net-(C4-Pad1)
- C4 pad 2: Net-(C4-Pad2) -> GND
- C5 pad 1: GND -> Net-(C5-Pad1)
- C5 pad 2: Net-(C5-Pad2) -> GND
- C6 pad 1: GND -> Net-(C6-Pad1)
- C6 pad 2: Net-(C6-Pad2) -> GND
- C7 pad 1: GND -> Net-(C7-Pad1)
- C7 pad 2: Net-(C7-Pad2) -> GND
- SW1 pad 1: Net-(C3-Pad2) -> Net-(C3-Pad1)
- SW2 pad 1: Net-(C4-Pad2) -> Net-(C4-Pad1)
- SW3 pad 1: Net-(C5-Pad2) -> Net-(C5-Pad1)
- SW4 pad 1: Net-(C6-Pad2) -> Net-(C6-Pad1)
- U3 pad 1: Net-(C7-Pad2) -> Net-(C7-Pad1)
Routing:
- net +12V: track 0.00 -> 18.7 mm
- net Net-(R6-Pad2): track 0.00 -> 18.2 mm
- net Net-(R5-Pad2): track 0.00 -> 18.2 mm
- net Net-(R4-Pad2): track 0.00 -> 18.2 mm
- net Net-(C7-Pad1): track 0.00 -> 18.1 mm
- net Net-(R3-Pad2): track 0.00 -> 17.9 mm
- net +5V: track 0.00 -> 16.1 mm
- net Net-(LED1-Pad2): track 0.00 -> 15.2 mm
- net Net-(BZ1-Pad1): track 0.00 -> 15.2 mm
- net Net-(C3-Pad1): track 0.00 -> 14.5 mm
- net Net-(C6-Pad1): track 0.00 -> 12.9 mm
- net Net-(C5-Pad1): track 0.00 -> 12.9 mm
- net Net-(J7-Pad1): track 0.00 -> 12.7 mm
- net Net-(J6-Pad1): track 0.00 -> 12.7 mm
- net Net-(J5-Pad1): track 0.00 -> 12.7 mm
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
Commit message: Started designing ing PCB 6
Other:
- board text added: "Devika Shaj, Gaadha P Nath, Shyama H, Athul T"

Commit message: Plotted gerber files for initial idea
Parts:
- added REF**: KiCad-Logo_5mm_Copper, Symbol:KiCad-Logo_5mm_Copper, F.Cu at (24.1, 17.8)
- moved REF** 7.62 mm to (266.7, 156.2)
- moved Pot4 3.81 mm to (180.3, 157.5)
- moved J2 1.27 mm to (21.6, 30.5)
Routing:
- net +5V: track 16.1 -> 227.0 mm
- net +12V: track 18.7 -> 54.3 mm
Other:
- board size 271.8 x 161.3 mm -> 270.5 x 162.6 mm

Commit message: Plotted gerber files for initial idea3
Parts:
- removed REF**: KiCad-Logo_5mm_Copper, Symbol:KiCad-Logo_5mm_Copper
- removed REF**: OSHW-Logo2_14.6x12mm_Copper, Symbol:OSHW-Logo2_14.6x12mm_Copper
- removed REF**: KiCad-Logo2_6mm_SilkScreen, Symbol:KiCad-Logo2_6mm_SilkScreen
- added R7: 4.7k, Resistor_THT:R_Axial_DIN0204_L3.6mm_D1.6mm_P5.08mm_Horizontal, F.Cu at (154.9, 16.5)
Connections:
- U2 pad 16: (no net) -> Net-(R7-Pad2)
Routing:
- net +5V: track 227.0 -> 310.1 mm
- net Net-(R7-Pad2): track 0.00 -> 65.5 mm

Commit message: PCB update with LCD 16x2
Parts:
- removed U2: NHD-0420H1Z, Display:NHD-0420H1Z
- added DS1: HY1602E, Display:HY1602E, F.Cu at (163.8, 26.7)
- added REF**: OSHW-Logo_11.4x12mm_Copper, Symbol:OSHW-Logo_11.4x12mm_Copper, F.Cu at (270.5, 154.9)
- added REF**: KiCad-Logo_8mm_Copper, Symbol:KiCad-Logo_8mm_Copper, F.Cu at (27.9, 21.6)
- added REF**: KiCad-Logo2_8mm_SilkScreen, Symbol:KiCad-Logo2_8mm_SilkScreen, F.Cu at (148.6, 95.2)
- R1, R2, R3, R4, R5, R6, R7: footprint Resistor_THT:R_Axial_DIN0204_L3.6mm_D1.6mm_P5.08mm_Horizontal -> Resistor_THT:R_Axial_DIN0207_L6.3mm_D2.5mm_P10.16mm_Horizontal
- moved BZ1 22.9 mm to (237.5, 26.7)
- moved J7 22.9 mm to (273.1, 54.6)
- moved LED1 22.9 mm to (265.4, 26.7)
- moved R1 22.9 mm to (237.5, 41.9)
- moved R2 22.9 mm to (268.0, 41.9)
- moved J6 22.9 mm to (242.6, 54.6)
- moved C2 20.5 mm to (74.9, 52.1)
- moved C1 19.3 mm to (45.7, 50.8)
- moved U1 18.8 mm to (55.9, 39.4)
- moved J2 7.62 mm to (21.6, 38.1)
- moved R7 3.81 mm to (154.9, 20.3)
- moved SW2 1.27 mm to (48.3, 153.7)
Routing:
- net Net-(DS1-Pad2): track 65.5 -> 8.67 mm
- net +5V: track 310.1 -> 338.5 mm
- net +12V: track 54.3 -> 49.2 mm
- net Net-(R3-Pad2): track 17.9 -> 21.5 mm
- net Net-(J6-Pad1): track 12.7 -> 14.8 mm
- net Net-(J7-Pad1): track 12.7 -> 14.8 mm
- net Net-(C3-Pad1): track 14.5 -> 13.0 mm
- net Net-(R4-Pad2): track 18.2 -> 19.4 mm
- net Net-(R5-Pad2): track 18.2 -> 19.4 mm
- net Net-(R6-Pad2): track 18.2 -> 19.4 mm
- net Net-(C5-Pad1): track 12.9 -> 12.1 mm
